File: swc.kicad_pcb (KiCad board)
At the start: 2 copper layers, 4 parts, among them IC1 LM2931CM, J1 Conn_02x03_Top_Bottom, U1 ATmega16M1-A, U2 TJA1043T

Commit message: Zamjenjen footprint
Parts:
- IC1: footprint KiCad:SOIC127P600X175-8N -> footprints:SOIC127P600X175-8N
Changed lines of the file:
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@@
 		)
 	)
-	(footprint "KiCad:SOIC127P600X175-8N"
+	(footprint "footprints:SOIC127P600X175-8N"
 		(layer "F.Cu")
 		(at 54.5 28.5)
@@
 			)
 		)
-		(property "Footprint" "SOIC127P600X175-8N"
+		(property "Footprint" "footprints:SOIC127P600X175-8N"
 			(at 0 0 0)
 			(unlocked yes)
@@
 		)
 		(fp_text user "${REFERENCE}"
-			(at 17.64 4.14 270)
-			(layer "F.Fab")
-			(effects
+			(at 17.64 4.14 -90)
+			(layer "F.Fab")
+			(effects
