File: swc.kicad_sch (KiCad schematic)
At the start: 4 parts, among them IC1 LM2931CM, J1 Conn_02x03_Top_Bottom, U1 ATmega16M1-A, U2 TJA1043T

Commit message: Zamjenjen footprint
Parts:
- IC1: footprint SOIC127P600X175-8N -> footprints:SOIC127P600X175-8N
Changed lines of the file:
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@@
 			)
 		)
-		(property "Footprint" "SOIC127P600X175-8N"
+		(property "Footprint" "footprints:SOIC127P600X175-8N"
 			(at 160.02 204.14 0)
 			(effects
